File: eagle/attiny_midi_cv.sch (EAGLE design)
At the start: 29 parts, among them IC1 TL072P, Q518 2N3904, U2 TINY45-20-DIP

Commit message: routed
Parts:
- removed CV_BUS_ENABLE, GATE_BUS_ENABLE: M02LOCK_LONGPADS, SparkFun-Connectors:M02LOCK_LONGPADS
- removed MIDI_IN_4: midi pin 4, wirepad:2,54/0,9
- removed MIDI_IN_5: midi pin 5, wirepad:2,54/0,9
- added MIDI_IN: 22-23-2021, con-molex:22-23-2021
- R26: device rcl:R-US_0207/7 -> rcl:R-US_0309/12
Connections:
- removed net N$1: GATE_BUS_ENABLE.2, PWR1.GATE
- removed net N$9: CV_BUS_ENABLE.2, PITCH.TIP, R10.2
- new net N$4: GATE.TIP, R26.1
- new net N$5: PITCH.TIP, R10.2
- net N$15: now also PITCH.NORM; no longer CV_BUS_ENABLE.1
- net N$25: now also U2.PB1(MISO); no longer U2.PB2(SCK/ADC1)
- net N$26: now also U2.PB0(MOSI); no longer U2.PB1(MISO)
- net N$3: now also MIDI_IN-2.S; no longer MIDI_IN_5.P
- net N$30: now also U2.PB3(ADC3); no longer U2.PB0(MOSI)
- net N$31: now also GATE.NORM, PWR1.GATE; no longer GATE.TIP, GATE_BUS_ENABLE.1, R26.1
- net N$45: now also U2.PB2(SCK/ADC1); no longer U2.PB3(ADC3)
- net N$8: now also MIDI_IN-1.S; no longer MIDI_IN_4.P
Other:
- moved on the sheet: R2
